Commit message: update (till 06-007)

File: my_robot_description/urdf/common_properties.xacro (robot description, xacro)
@@ -12,3 +12,36 @@
         <color rgba="0.5 0.5 0.5 1.0"/>
     </material>
+    <xacro:macro name="box_inertia" params="m x y z o_xyz o_rpy">
+        <inertial>
+            <!-- Note! There is a "l" in "inertial" -->
+            <mass value="${m}"/>
+            <origin xyz="${o_xyz}" rpy="${o_rpy}"/>
+            <inertia
+                ixx="${(1/12.0) * m * (y**2 + z**2)}" ixy="0.0" ixz="0.0"
+                iyy="${(1/12.0) * m * (x**2 + z**2)}" iyz="0.0"
+                izz="${(1/12.0) * m * (x**2 + y**2)}"/>
+            <!-- The parameters are kinda different in wikipedia, and it can be confusing to follow the naming condition in wiki.
+            Just remember the inertia of one axis is calculated by the value of the other two axes. -->
+        </inertial>
+    </xacro:macro>
+    <xacro:macro name="cylinder_inertia" params="m r l o_xyz o_rpy">
+        <inertial>
+            <mass value="${m}"/>
+            <origin xyz="${o_xyz}" rpy="${o_rpy}"/>
+            <inertia
+                ixx="${(1/12.0) * m * (3 * r**2 + l**2)}" ixy="0.0" ixz="0.0"
+                iyy="${(1/12.0) * m * (3 * r**2 + l**2)}" iyz="0.0"
+                izz="${(1/2.0) * m * r**2}"/>
+        </inertial>
+    </xacro:macro>
+    <xacro:macro name="sphere_inertia" params="m r o_xyz o_rpy">
+        <inertial>
+            <mass value="${m}"/>
+            <origin xyz="${o_xyz}" rpy="${o_rpy}"/>
+            <inertia
+                ixx="${(2/5.0) * m * r**2}" ixy="0.0" ixz="0.0"
+                iyy="${(2/5.0) * m * r**2}" iyz="0.0"
+                izz="${(2/5.0) * m * r**2}"/>
+        </inertial>
+    </xacro:macro>
 </robot>

File: my_robot_description/urdf/mobile_base.xacro (robot description, xacro)
@@ -16,4 +16,15 @@
             <material name="blue"/>
         </visual>
+        <collision>
+            <geometry>
+                <box size="${base_length} ${base_width} ${base_height}"/>
+            </geometry>
+            <origin xyz="0 0 ${base_height / 2.0}" rpy="0 0 0"/>
+            <!-- quite the same as visual, no material though -->
+        </collision>
+        <xacro:box_inertia m="5.0" x="${base_length}" y="${base_width}" z="${base_height}"
+                           o_xyz="0 0 ${base_height / 2.0}" o_rpy="0 0 0"/>
+            <!-- The mass unit is kg -->
+            <!-- The origin xyz here is the same as the visual origin xyz. -->
     </link>
     <xacro:macro name="wheel_link" params="prefix">
@@ -26,4 +37,14 @@
                 <material name="gray" />
             </visual>
+            <collision>
+                <geometry>
+                    <sphere radius="${wheel_radius}" />
+                </geometry>
+                <origin xyz="0 0 0" rpy="0 0 0" />
+                <!-- here we use sphere instead of cylinder for collision to simplify the calculation -->
+                <!-- and the rpy doesn't matter any more in sphere -->
+            </collision>
+            <xacro:cylinder_inertia m="1.0" r="${wheel_radius}" l="${wheel_length}"
+                                    o_xyz="0 0 0" o_rpy="${pi / 2.0} 0 0"/>
         </link>
     </xacro:macro>
@@ -38,4 +59,12 @@
             <material name="gray" />
         </visual>
+        <collision>
+            <geometry>
+                <sphere radius="${wheel_radius / 2.0}" />
+            </geometry>
+            <origin xyz="0 0 0" rpy="0 0 0" />
+        </collision>
+        <xacro:sphere_inertia m="0.5" r="${wheel_radius / 2.0}"
+                              o_xyz="0 0 0" o_rpy="0 0 0"/>
     </link>
     <link name="base_footprint">
