Commit message: update (till moveit 05-005)

File: my_robot_2_description/urdf/arm.xacro (robot description, xacro)
@@ -106,6 +106,5 @@
         </collision>
     </link>
-    <link name="tool_link">
-    </link>
+    <link name="tool_link" />
     <joint name="joint1" type="revolute">
         <parent link="base_link"/>

File: my_robot_2_description/urdf/common_properties.xacro (robot description, xacro)
@@ -7,3 +7,9 @@
         <color rgba="0 0 0.5 1.0"/>
     </material>
+    <material name="dark_green">
+        <color rgba="0 0.4 0 1" />
+    </material>
+    <material name="light_green">
+        <color rgba="0 0.6 0 1" />
+    </material>
 </robot>

File: my_robot_2_description/urdf/my_robot_2.urdf.xacro (robot description, xacro)
@@ -3,3 +3,9 @@
     <xacro:include filename="common_properties.xacro" />
     <xacro:include filename="arm.xacro" />
+    <xacro:include filename="gripper.xacro" />
+    <joint name="gripper_base_joint" type="fixed">
+        <parent link="tool_link" />
+        <child link="gripper_base_link" />
+        <origin xyz="0 0 0" rpy="0 0 0" />
+    </joint>
 </robot>

File: my_robot_moveit_config/config/my_robot_2.ros2_control.xacro (robot description, xacro)
@@ -44,4 +44,10 @@
                 </state_interface>
             </joint>
+            <joint name="gripper_left_finger_joint">
+                <command_interface name="position"/>
+                <state_interface name="position">
+                  <param name="initial_value">${initial_positions['gripper_left_finger_joint']}</param>
+                </state_interface>
+            </joint>
         </ros2_control>
     </xacro:macro>
